File: TFPilot01A/hw/sch_pcb/CPU.sch (KiCad schematic (older format))
At the start: 1 part

Commit message: Kreslení schéma
Parts:
- added C? (x10): 100nF, Mlab_R:SMD-0603, symbol Device:C
- added C? (x2): 8pF, symbol Device:C
- added C? (x3): 2u2F, symbol Device:C
- added R? (x4): 0R, Mlab_R:SMD-0603, symbol Device:R
- added R?: 1M, symbol Device:R
- added R? (x2): 10k, symbol Device:R
- added R?: 10k, Mlab_R:SMD-0603, symbol Device:R
- added SW?: TACTM-64M-F, Button_Switch_THT:SW_PUSH_6mm_H4.3mm, symbol Switch:SW_Push
- added U?: REF3333AIDCKT, Package_TO_SOT_SMD:SOT-23, symbol Reference_Voltage:REF3033
- added Y?: NX3225SA-16MHZ-STD-CSR-6, symbol Device:Crystal_GND24
Connections:
- net GND: now reaches U?.102 (VSS)
- net GND: now also U?.113 (VSS), U?.126 (VSS), U?.135 (VSS), U?.14 (VSS), U?.148 (VSS), U?.158 (VSS), U?.22 (VSS), U?.48 (BYPASS_REG), U?.61 (VSS), U?.71 (VSS), U?.90 (VSS), C?.1, C?.1, C?.1, C?.1, C?.2, C?.2, C?.2, C?.2, C?.2, C?.2, C?.2, C?.2, C?.2, C?.2, C?.2, R?.1, R?.2, R?.2, R?.2, Y?.2, Y?.4
- net at U?.103 (VDD): now also U?.127 (VDD), U?.136 (VDD), U?.149 (VDDSDMMC), U?.15 (VDD), U?.159 (VDD), U?.172 (VDD), U?.23 (VDD), U?.36 (VDD), U?.49 (VDD), U?.62 (VDD), U?.72 (VDD), U?.82 (VDD), U?.91 (VDD), R?.1
- net MCU_3V3: now reaches U?.114 (VDDUSB)
- net MCU_3V3: now also C?.1, C?.1, C?.1, C?.1, C?.1, C?.1, C?.1, R?.1, R?.1, SW?.2
- net at U?.125 (VCAP_2): now also C?.2
- net BOOT0: now reaches U?.166 (BOOT0)
- net BOOT0: now also R?.2, SW?.1
- net PDR_ON: now reaches U?.171 (PDR_ON)
- net PDR_ON: now also R?.1, R?.2
- net at U?.29 (PH0): now also C?.2, R?.1, Y?.3
- net at U?.30 (PH1): now also C?.2, R?.2, Y?.1
- net at U?.31 (NRST): now also R?.2
- net VSSA: now reaches U?.37 (VSSA)
- net VSSA: now also R?.1
- net VREF+: now reaches U?.38 (VREF+)
- net VREF+: now also C?.1, C?.1, U?.2 (OUT)
- net AVDD: now reaches U?.39 (VDDA)
- net AVDD: now also C?.1, R?.2
- net VBAT: now reaches U?.6 (VBAT)
- net at U?.81 (VCAP_1): now also C?.2
- new net: R?.1, U?.3 (GND)
- new net VDD_5V_IN: C?.1, U?.1 (IN)
